Commit message: update workspace to add collision object

File: ur-sim/ur_sim/assets/ur3e_workspace/workspace.urdf (robot description, URDF)
Before this commit: robot workspace.urdf, 1 links, 0 joints
Links:
- link baseLink: geometry collision box size=1 0.5 0.01; visual mesh filename=plane.obj scale=1 0.5 1

Commit message: some finetuning on joints for UR

File: ur-sim/ur_sim/assets/ur3e_workspace/workspace.urdf (robot description, URDF)
Before this commit: robot workspace.urdf, 1 links, 0 joints
Links:
- link baseLink: geometry collision box size=1 1 0.01; visual mesh filename=plane.obj scale=1 0.5 1
