Commit message: lock

File: pybullet-sim/pybullet_sim/assets/robotiq2f85/robotiq_2f_85.urdf (robot description, URDF)
Before this commit: robot robotiq_2f-85, 11 links, 10 joints
Joints:
- joint left_inner_finger_joint: mimic joint=finger_joint multiplier=-1 offset=0 -> (none)
- joint left_inner_knuckle_joint: mimic joint=finger_joint multiplier=1 offset=0 -> (none)
- joint right_inner_finger_joint: mimic joint=finger_joint multiplier=-1 offset=0 -> (none)
- joint right_inner_knuckle_joint: mimic joint=finger_joint multiplier=1 offset=0 -> (none)
- joint right_outer_knuckle_joint: mimic joint=finger_joint multiplier=1 offset=0 -> (none)

Commit message: found culprit: finger tip masses were set to 1kg!

File: pybullet-sim/pybullet_sim/assets/robotiq2f85/robotiq_2f_85.urdf (robot description, URDF)
Before this commit: robot robotiq_2f-85, 11 links, 10 joints
Links:
- link left_inner_finger_pad: mass 1. -> 0.01
- link right_inner_finger_pad: mass 1 -> 0.01
- link robotiq_arg2f_base_link: mass 0.22652 -> 1.0

Commit message: gripper - robot init order seems to matter??

File: pybullet-sim/pybullet_sim/assets/robotiq2f85/robotiq_2f_85.urdf (robot description, URDF)
Before this commit: robot robotiq_2f-85, 11 links, 10 joints
Links:
- link left_inner_finger_pad: geometry collision box size=0.022 0.00635 0.0375; visual box size=0.022 0.00635 0.0375
- link right_inner_finger_pad: geometry collision box size=0.022 0.00635 0.0375; visual box size=0.022 0.00635 0.0375
